Commit message: update joint limits

File: kinova_2f_lite_description/urdf/kinova_2f_lite_macro.urdf.xacro (robot description, xacro)
@@ -110,6 +110,6 @@
         </link>
         <joint name="${prefix}right_finger_tip_joint" type="revolute">
-            <!-- <mimic joint="${prefix}right_finger_bottom_joint" multiplier="-0.676" offset="0.149" /> -->
-            <mimic joint="${prefix}right_finger_bottom_joint" multiplier="-0.276" offset="-0.1" />
+            <mimic joint="${prefix}right_finger_bottom_joint" multiplier="-0.676" offset="0.149" />
+            <!-- <mimic joint="${prefix}right_finger_bottom_joint" multiplier="-0.276" offset="-0.1" /> -->
             <origin rpy="0 0 0" xyz="-0.045636 0.020423 0" />
             <parent link="${prefix}right_finger_prox_link" />
@@ -146,10 +146,10 @@
         </link>
         <joint name="${prefix}left_finger_bottom_joint" type="revolute">
-            <mimic joint="${prefix}right_finger_bottom_joint" multiplier="-1.0" offset="0.0" />
+            <mimic joint="${prefix}right_finger_bottom_joint" multiplier="1.0" offset="0.0" />
             <origin xyz="0 0.0305 0.070003" rpy="-1.571 0.611 -1.571" />
             <!-- <origin rpy="0 1.5708 0" xyz="0 0.0305 0.070003" /> -->
             <parent link="${prefix}gripper_base_link" />
             <child link="${prefix}left_finger_prox_link" />
-            <axis xyz="0 0 -1" />
+            <axis xyz="0 0 1" />
             <limit lower="${min_left_finger_bottom_joint_pos}" upper="${max_left_finger_bottom_joint_pos}"
                     effort="${left_finger_bottom_joint_effort}" velocity="${left_finger_bottom_joint_vel}" />
@@ -182,6 +182,6 @@
         </link>
         <joint name="${prefix}left_finger_tip_joint" type="revolute">
-            <!-- <mimic joint="${prefix}right_finger_bottom_joint" multiplier="-0.676" offset="0.149" /> -->
-            <mimic joint="${prefix}right_finger_bottom_joint" multiplier="-0.276" offset="-0.1" />
+            <mimic joint="${prefix}right_finger_bottom_joint" multiplier="-0.676" offset="0.149" />
+            <!-- <mimic joint="${prefix}right_finger_bottom_joint" multiplier="-0.276" offset="-0.1" /> -->
             <origin rpy="0 0 0" xyz="-0.045636 -0.020423 6.9901E-05" />
             <parent link="${prefix}left_finger_prox_link" />

Commit message: update limits

File: kinova_2f_lite_description/urdf/kinova_2f_lite_macro.urdf.xacro (robot description, xacro)
@@ -110,6 +110,6 @@
         </link>
         <joint name="${prefix}right_finger_tip_joint" type="revolute">
-            <mimic joint="${prefix}right_finger_bottom_joint" multiplier="-0.676" offset="0.149" />
-            <!-- <mimic joint="${prefix}right_finger_bottom_joint" multiplier="-0.276" offset="-0.1" /> -->
+            <!-- <mimic joint="${prefix}right_finger_bottom_joint" multiplier="-0.676" offset="0.149" /> -->
+            <mimic joint="${prefix}right_finger_bottom_joint" multiplier="-0.276" offset="-0.1" />
             <origin rpy="0 0 0" xyz="-0.045636 0.020423 0" />
             <parent link="${prefix}right_finger_prox_link" />
@@ -146,10 +146,10 @@
         </link>
         <joint name="${prefix}left_finger_bottom_joint" type="revolute">
-            <mimic joint="${prefix}right_finger_bottom_joint" multiplier="1.0" offset="0.0" />
+            <mimic joint="${prefix}right_finger_bottom_joint" multiplier="-1.0" offset="0.0" />
             <origin xyz="0 0.0305 0.070003" rpy="-1.571 0.611 -1.571" />
             <!-- <origin rpy="0 1.5708 0" xyz="0 0.0305 0.070003" /> -->
             <parent link="${prefix}gripper_base_link" />
             <child link="${prefix}left_finger_prox_link" />
-            <axis xyz="0 0 1" />
+            <axis xyz="0 0 -1" />
             <limit lower="${min_left_finger_bottom_joint_pos}" upper="${max_left_finger_bottom_joint_pos}"
                     effort="${left_finger_bottom_joint_effort}" velocity="${left_finger_bottom_joint_vel}" />
@@ -182,6 +182,6 @@
         </link>
         <joint name="${prefix}left_finger_tip_joint" type="revolute">
-            <mimic joint="${prefix}right_finger_bottom_joint" multiplier="-0.676" offset="0.149" />
-            <!-- <mimic joint="${prefix}right_finger_bottom_joint" multiplier="-0.276" offset="-0.1" /> -->
+            <!-- <mimic joint="${prefix}right_finger_bottom_joint" multiplier="-0.676" offset="0.149" /> -->
+            <mimic joint="${prefix}right_finger_bottom_joint" multiplier="-0.276" offset="-0.1" />
             <origin rpy="0 0 0" xyz="-0.045636 -0.020423 6.9901E-05" />
             <parent link="${prefix}left_finger_prox_link" />
